File: _saved_pocketbone-kicad.sch (KiCad schematic (older format))
At the start: 91 parts, among them P1 USB_OTG, P2 USB_OTG, P3 CONN_01X10, P4 CONN_02X02, SW1 SW_PUSH_SMALL_H, SW2 SW_PUSH_SMALL_H, U1 SN74LVC1G07, U2 OSD3358, U3 24LC32AT-I/OT, U4 TPS2051C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

Commit message: wip
Parts:
- C20, C22, C23: renamed from C?; footprint Capacitors_SMD:C_0402 -> Capacitor_SMD:C_0402_1005Metric
- C21: renamed from C?; footprint Capacitors_SMD:C_0402 -> Capacitor_SMD:C_0201_0603Metric
- J1, J2, J3, J4: renamed from J?; footprint (none) -> Connector_JST:JST_GH_BM04B-GHS-TBT_1x04-1MP_P1.25mm_Vertical
- J5, J6: renamed from J?; footprint (none) -> Connector_PinHeader_2.00mm:PinHeader_1x10_P2.00mm_Vertical_SMD_Pin1Left
- gave numbers to parts that had none: 19
